Commit message: Reward Copleted

File: RL_SPIDER/Simulator/catkin_ws/rl_spider/urdf/spider.xacro (robot description, xacro)
@@ -4,9 +4,10 @@
 	<xacro:property name="len_2" value="0.3" />
 	<xacro:property name="len_3" value="0.35" />
+	<xacro:property name="cyl_name" value="a" />
 	<xacro:property name="rad" value="0.1" />
 	<xacro:property name="pi" value="3.1457" />
 	<xacro:property name="len_sq" value="0.4" />
 	<xacro:macro name="leg" params="cyl_num">
-		<link name="${cyl_num}">
+		<link name="${cyl_name}+'d'">
 			<visual>
 				<geometry>
@@ -18,22 +19,4 @@
 				</material>
 			</visual>
-			<visual>
-				<geometry>
-					<sphere radius="${rad}"/>
-				</geometry>
-				<origin rpy="0 0 0" xyz="${len_1/2.828427125} ${len_1/2.828427125} 0"/>
-				<material name="yellow">
-					<color rgba="0 1 1 1"/>
-				</material>
-			</visual>
-			<visual>
-				<geometry>
-					<sphere radius="${rad}"/>
-				</geometry>
-				<origin rpy="0 0 0" xyz="${len_1/-2.828427125} ${len_1/-2.828427125} 0"/>
-				<material name="yellow">
-					<color rgba="0 1 1 1"/>
-				</material>
-			</visual>
 		</link>
 	</xacro:macro>
